Commit message: add sonar sensor + fix buoyancy robot

File: urdf/robot.xacro (robot description, xacro)
@@ -3,5 +3,5 @@
   <link name="base_link">
     <visual>
-      <origin rpy="0 0 0" xyz="0 0 -0.95" />
+      <origin rpy="0 0 0" xyz="0 0 0" />
       <geometry>
         <mesh filename="package://robot-lab/meshes/robot.dae" />
@@ -9,5 +9,5 @@
     </visual>
     <collision>
-      <origin rpy="0 0 0" xyz="0 0 -0.95" />
+      <origin rpy="0 0 0" xyz="0 0 0" />
       <geometry>
         <mesh filename="package://robot-lab/meshes/robot.dae" />
@@ -15,6 +15,6 @@
     </collision>
     <inertial>
-      <mass value="38.45735" />
-      <origin xyz="0 0 -0.95" />
+      <mass value="37.5000" />
+      <origin xyz="0 0 -0.9" />
       <inertia ixx="1" ixy="0.0" ixz="0.0" iyy="1" iyz="0.0" izz="1" />
     </inertial>
@@ -35,3 +35,64 @@
     </plugin>
   </gazebo>
+  <joint name="sonar_joint" type="fixed">
+    <parent link="base_link" />
+    <child link="sonar_link" />
+    <origin xyz="0.334 0 0.06" />
+  </joint>
+  <link name="sonar_link">
+    <inertial>
+      <mass value="0.001" />
+      <origin xyz="0 0 0" rpy="0 0 0" />
+      <inertia ixx="0.000000017" ixy="0" ixz="0" iyy="0.000000017" iyz="0" izz="0.000000017" />
+    </inertial>
+    <visual>
+      <origin xyz="0 0 0" rpy="0 0 0" />
+      <geometry>
+        <mesh filename="package://robot-lab/meshes/max_sonar_ez4.dae" />
+      </geometry>
+    </visual>
+    <collision>
+      <origin xyz="0 0 0" rpy="0 0 0" />
+      <geometry>
+        <box size="0.01 0.01 0.01" />
+      </geometry>
+    </collision>
+  </link>
+  <gazebo reference="sonar_link">
+    <sensor type="ray" name="sonar">
+      <pose>0 0 0 0 0 0</pose>
+      <visualize>true</visualize>
+      <update_rate>50</update_rate>
+      <ray>
+        <scan>
+          <horizontal>
+            <samples>10</samples>
+            <resolution>1</resolution>
+            <min_angle>-0.14835</min_angle>
+            <max_angle>0.14835</max_angle>
+          </horizontal>
+          <vertical>
+            <samples>10</samples>
+            <resolution>1</resolution>
+            <min_angle>-0.14835</min_angle>
+            <max_angle>0.14835</max_angle>
+          </vertical>
+        </scan>
+        <range>
+          <min>0.01</min>
+          <max>3</max>
+          <resolution>0.02</resolution>
+        </range>
+      </ray>
+      <plugin filename="libgazebo_ros_range.so" name="gazebo_ros_range">
+        <gaussianNoise>0.005</gaussianNoise>
+        <alwaysOn>true</alwaysOn>
+        <updateRate>50</updateRate>
+        <topicName>sonar</topicName>
+        <frameName>sonar_link</frameName>
+        <radiation>INFRARED</radiation>
+        <fov>0.2967</fov>
+      </plugin>
+    </sensor>
+  </gazebo>
 </robot>

Commit message: add camera rgb

File: urdf/robot.xacro (robot description, xacro)
@@ -96,3 +96,66 @@
     </sensor>
   </gazebo>
+  <joint name="camera_joint" type="fixed">
+    <axis xyz="0 1 0" />
+    <origin xyz="0.25 0 0.12" rpy="0 0 0" />
+    <parent link="base_link" />
+    <child link="camera_link" />
+  </joint>
+  <!-- Camera -->
+  <link name="camera_link">
+    <collision>
+      <origin xyz="0 0 0" rpy="0 0 0" />
+      <geometry>
+        <mesh filename="package://robot-lab/meshes/flir_a35_housing.stl" />
+      </geometry>
+    </collision>
+    <visual>
+      <origin xyz="0 0 0" rpy="0 0 0" />
+      <geometry>
+        <mesh filename="package://robot-lab/meshes/flir_a35_housing.stl" />
+      </geometry>
+    </visual>
+    <inertial>
+      <mass value="1e-5" />
+      <origin xyz="0 0 0" rpy="0 0 0" />
+      <inertia ixx="1e-6" ixy="0" ixz="0" iyy="1e-6" iyz="0" izz="1e-6" />
+    </inertial>
+  </link>
+  <!-- camera -->
+  <gazebo reference="camera_link">
+    <sensor type="camera" name="camera1">
+      <update_rate>30.0</update_rate>
+      <camera name="head">
+        <horizontal_fov>1.3962634</horizontal_fov>
+        <image>
+          <width>800</width>
+          <height>800</height>
+          <format>R8G8B8</format>
+        </image>
+        <clip>
+          <near>0.02</near>
+          <far>300</far>
+        </clip>
+        <noise>
+          <type>gaussian</type>
+          <mean>0.0</mean>
+          <stddev>0.007</stddev>
+        </noise>
+      </camera>
+      <plugin name="camera_controller" filename="libgazebo_ros_camera.so">
+        <alwaysOn>true</alwaysOn>
+        <updateRate>0.0</updateRate>
+        <cameraName>rrbot/camera1</cameraName>
+        <imageTopicName>image_raw</imageTopicName>
+        <cameraInfoTopicName>camera_info</cameraInfoTopicName>
+        <frameName>camera_link</frameName>
+        <hackBaseline>0.07</hackBaseline>
+        <distortionK1>0.0</distortionK1>
+        <distortionK2>0.0</distortionK2>
+        <distortionK3>0.0</distortionK3>
+        <distortionT1>0.0</distortionT1>
+        <distortionT2>0.0</distortionT2>
+      </plugin>
+    </sensor>
+  </gazebo>
 </robot>

Commit message: add cliff rocks into ocean world

File: urdf/robot.xacro (robot description, xacro)
@@ -20,24 +20,4 @@
     </inertial>
   </link>
-  <gazebo>
-    <plugin name="BuoyancyPlugin" filename="libBuoyancyPlugin.so">
-      <fluid_density>1000</fluid_density>
-    </plugin>
-  </gazebo>
-  <gazebo>
-    <plugin name="omni_steering" filename="libgazebo_ros_planar_move.so">
-      <commandTopic>cmd_vel</commandTopic>
-      <odometryTopic>odom</odometryTopic>
-      <codometryFrame>odom</codometryFrame>
-      <codometryRate>50.0</codometryRate>
-      <robotBaseFrame>base_link</robotBaseFrame>
-      <publishTF>false</publishTF>
-    </plugin>
-  </gazebo>
-  <joint name="sonar_joint" type="fixed">
-    <parent link="base_link" />
-    <child link="sonar_link" />
-    <origin xyz="0.334 0 0.06" />
-  </joint>
   <link name="sonar_link">
     <inertial>
@@ -59,4 +39,25 @@
     </collision>
   </link>
+  <link name="camera_link">
+    <collision>
+      <origin xyz="0 0 0" rpy="0 0 0" />
+      <geometry>
+        <mesh filename="package://robot-lab/meshes/flir_a35_housing.stl" />
+      </geometry>
+    </collision>
+    <visual>
+      <origin xyz="0 0 0" rpy="0 0 0" />
+      <geometry>
+        <mesh filename="package://robot-lab/meshes/flir_a35_housing.stl" />
+      </geometry>
+    </visual>
+    <inertial>
+      <mass value="1e-5" />
+      <origin xyz="0 0 0" rpy="0 0 0" />
+      <inertia ixx="1e-6" ixy="0" ixz="0" iyy="1e-6" iyz="0" izz="1e-6" />
+    </inertial>
+  </link>
+  <!-- SENSORS -->
+  <!-- SONAR -->
   <gazebo reference="sonar_link">
     <sensor type="ray" name="sonar">
@@ -91,36 +92,10 @@
         <topicName>sonar</topicName>
         <frameName>sonar_link</frameName>
-        <radiation>INFRARED</radiation>
+        <radiation>ULTRASOUND</radiation>
         <fov>0.2967</fov>
       </plugin>
     </sensor>
   </gazebo>
-  <joint name="camera_joint" type="fixed">
-    <axis xyz="0 1 0" />
-    <origin xyz="0.25 0 0.12" rpy="0 0 0" />
-    <parent link="base_link" />
-    <child link="camera_link" />
-  </joint>
-  <!-- Camera -->
-  <link name="camera_link">
-    <collision>
-      <origin xyz="0 0 0" rpy="0 0 0" />
-      <geometry>
-        <mesh filename="package://robot-lab/meshes/flir_a35_housing.stl" />
-      </geometry>
-    </collision>
-    <visual>
-      <origin xyz="0 0 0" rpy="0 0 0" />
-      <geometry>
-        <mesh filename="package://robot-lab/meshes/flir_a35_housing.stl" />
-      </geometry>
-    </visual>
-    <inertial>
-      <mass value="1e-5" />
-      <origin xyz="0 0 0" rpy="0 0 0" />
-      <inertia ixx="1e-6" ixy="0" ixz="0" iyy="1e-6" iyz="0" izz="1e-6" />
-    </inertial>
-  </link>
-  <!-- camera -->
+  <!-- CAMERA -->
   <gazebo reference="camera_link">
     <sensor type="camera" name="camera1">
@@ -159,3 +134,31 @@
     </sensor>
   </gazebo>
+  <!-- PLUGINS -->
+  <gazebo>
+    <plugin name="BuoyancyPlugin" filename="libBuoyancyPlugin.so">
+      <fluid_density>1000</fluid_density>
+    </plugin>
+  </gazebo>
+  <gazebo>
+    <plugin name="omni_steering" filename="libgazebo_ros_planar_move.so">
+      <commandTopic>cmd_vel</commandTopic>
+      <odometryTopic>odom</odometryTopic>
+      <codometryFrame>odom</codometryFrame>
+      <codometryRate>50.0</codometryRate>
+      <robotBaseFrame>base_link</robotBaseFrame>
+      <publishTF>false</publishTF>
+    </plugin>
+  </gazebo>
+  <!-- JOINTS -->
+  <joint name="sonar_joint" type="fixed">
+    <parent link="base_link" />
+    <child link="sonar_link" />
+    <origin xyz="0.334 0 0.06" />
+  </joint>
+  <joint name="camera_joint" type="fixed">
+    <axis xyz="0 1 0" />
+    <origin xyz="0.25 0 0.12" rpy="0 0 0" />
+    <parent link="base_link" />
+    <child link="camera_link" />
+  </joint>
 </robot>

Commit message: implementation bug2 algorithm

File: urdf/robot.xacro (robot description, xacro)
@@ -20,5 +20,5 @@
     </inertial>
   </link>
-  <link name="sonar_link">
+  <link name="hokuyo_link">
     <inertial>
       <mass value="0.001" />
@@ -59,4 +59,35 @@
   </link>
   <!-- SENSORS -->
+  <gazebo reference="hokuyo_link">
+    <sensor type="ray" name="head_hokuyo_sensor">
+      <pose>0 0 0 0 0 0</pose>
+      <visualize>true</visualize>
+      <update_rate>100</update_rate>
+      <ray>
+        <scan>
+          <horizontal>
+            <samples>720</samples>
+            <resolution>1</resolution>
+            <min_angle>-2</min_angle>
+            <max_angle>2</max_angle>
+          </horizontal>
+        </scan>
+        <range>
+          <min>0.1</min>
+          <max>5.6</max>
+          <resolution>0.01</resolution>
+        </range>
+        <noise>
+          <type>gaussian</type>
+          <mean>0.0</mean>
+          <stddev>0.01</stddev>
+        </noise>
+      </ray>
+      <plugin name="gazebo_ros_head_hokuyo_controller" filename="libgazebo_ros_laser.so">
+        <topicName>/rrbot/laser/scan</topicName>
+        <frameName>hokuyo_link</frameName>
+      </plugin>
+    </sensor>
+  </gazebo>
   <!-- SONAR -->
   <gazebo reference="sonar_link">
@@ -153,5 +184,5 @@
   <joint name="sonar_joint" type="fixed">
     <parent link="base_link" />
-    <child link="sonar_link" />
+    <child link="hokuyo_link" />
     <origin xyz="0.334 0 0.06" />
   </joint>
