Commit message: fixs

File: description/urdf/argo.gazebo.xacro (robot description, xacro)
@@ -8,5 +8,5 @@
   <xacro:macro name="argo_hydro_model" params="namespace">
     <link name="${namespace}/base_link">
-      <neutrally_buoyant>1</neutrally_buoyant>
+      <neutrally_buoyant>0</neutrally_buoyant>
       <volume>${volume}</volume>
       <box>
@@ -16,4 +16,7 @@
       </box>
       <center_of_buoyancy>${cob}</center_of_buoyancy>
+      <!-- <metacentric_width>0.4</metacentric_width>
+      <metacentric_length>0.4</metacentric_length>
+      <water_level_plane_area>0.48</water_level_plane_area> -->
       <hydrodynamic_model>
         <type>fossen</type>

File: description/urdf/argo_actuators.xacro (robot description, xacro)
@@ -2,11 +2,11 @@
 <robot xmlns:xacro="http://www.ros.org/wiki/xacro">
   <xacro:thruster_macro namespace="${namespace}" thruster_id="0">
-    <origin xyz="-0.088 -0.1192 -0.0061828" rpy="0 0 ${pi}" />
+    <origin xyz="-0.25 -0.1192 -0.0061828" rpy="0 0 ${pi}" />
   </xacro:thruster_macro>
   <xacro:thruster_macro namespace="${namespace}" thruster_id="1">
-    <origin xyz="-0.088 0.1192 -0.0061828" rpy="0 0 ${pi}" />
+    <origin xyz="-0.25 0.1192 -0.0061828" rpy="0 0 ${pi}" />
   </xacro:thruster_macro>
-  <xacro:thruster_macro namespace="${namespace}" thruster_id="2">
-    <origin xyz="0.067 0 0.1258172" rpy="0 -${0.5*pi} 0" />
-  </xacro:thruster_macro>
+  <!-- <xacro:thruster_macro namespace="${namespace}" thruster_id="2">
+    <origin xyz="0.1 0 0.1258172" rpy="0 -${0.5*pi} 0" />
+  </xacro:thruster_macro> -->
 </robot>

File: description/urdf/argo_sensors.xacro (robot description, xacro)
@@ -1,53 +1,35 @@
 <?xml version="1.0"?>
 <robot xmlns:xacro="http://www.ros.org/wiki/xacro">
+  <!-- Mount a camera -->
+  <xacro:default_camera namespace="${namespace}" parent_link="${namespace}/base_link" suffix="">
+    <origin xyz="0.55 0.0025 0.12" rpy="0 0 0" />
+  </xacro:default_camera>
   <!-- Mount a GPS. -->
   <xacro:default_gps namespace="${namespace}" parent_link="${namespace}/base_link" />
   <!-- Mount a Pose 3D sensor. -->
   <xacro:default_pose_3d_macro namespace="${namespace}" parent_link="${namespace}/base_link" inertial_reference_frame="${inertial_reference_frame}" />
-  <!-- IMU  -->
-  <xacro:default_imu_macro namespace="${namespace}" parent_link="${namespace}/base_link" inertial_reference_frame="${inertial_reference_frame}">
-    <origin xyz="0 0 0" rpy="0 0 0" />
-  </xacro:default_imu_macro>
-  <!-- Add a chemical particle concentration sensor -->
-  <xacro:default_chemical_concentration_sensor namespace="${namespace}" parent_link="${namespace}/base_link">
-    <origin xyz="0 0 0" rpy="0 0 0" />
-  </xacro:default_chemical_concentration_sensor>
-  <!-- DVL  -->
-  <!-- <xacro:default_dvl_macro namespace="${namespace}" parent_link="${namespace}/base_link" inertial_reference_frame="${inertial_reference_frame}">
-    <origin xyz="0.294307 0.468494 -0.68" rpy="0 ${0.5*pi} 0" />
-  </xacro:default_dvl_macro> -->
-  <!-- Magnetometer  -->
-  <!-- <xacro:default_magnetometer namespace="${namespace}" parent_link="${namespace}/base_link" /> -->
-  <!-- RPT  -->
-  <!-- <xacro:default_rpt namespace="${namespace}" parent_link="${namespace}/base_link">
-    <origin xyz="-1.32 0 0.8" rpy="0 0 0" />
-  </xacro:default_rpt> -->
-  <!-- Pressure  -->
-  <!-- <xacro:default_pressure_macro namespace="${namespace}" parent_link="${namespace}/base_link">
-    <origin xyz="-1.32 0.5 0.85" rpy="0 0 0" />
-  </xacro:default_pressure_macro> -->
-  <!-- IMU  -->
-  <!-- <xacro:default_imu_macro namespace="${namespace}" parent_link="${namespace}/base_link" inertial_reference_frame="${inertial_reference_frame}">
-    <origin xyz="0 0 0" rpy="0 0 0" />
-  </xacro:default_imu_macro> -->
-  <!-- Mount a camera -->
-  <!-- <xacro:default_camera namespace="${namespace}" parent_link="${namespace}/base_link" suffix="">
-    <origin xyz="1.15 0 0.4" rpy="0 0.6 0" />
-  </xacro:default_camera> -->
-  <!-- <xacro:default_camera namespace="${namespace}" parent_link="${namespace}/base_link" suffix="right">
-    <origin xyz="1.15 -0.63 0.4" rpy="0 0.6 0.4" />
-  </xacro:default_camera> -->
-  <!-- <xacro:default_camera namespace="${namespace}" parent_link="${namespace}/base_link" suffix="left">
-    <origin xyz="1.15 0.63 0.4" rpy="0 0.6 -0.4" />
-  </xacro:default_camera> -->
-  <!-- Mount a GPS. -->
-  <!-- <xacro:default_gps namespace="${namespace}" parent_link="${namespace}/base_link" /> -->
-  <!-- Mount a Pose 3D sensor. -->
-  <!-- <xacro:default_pose_3d_macro namespace="${namespace}" parent_link="${namespace}/base_link" inertial_reference_frame="${inertial_reference_frame}" /> -->
-  <!-- Mount chemical particle concentration sensor -->
-  <!-- <xacro:default_chemical_concentration_sensor_macro namespace="${namespace}" parent_link="${namespace}/base_link" inertial_reference_frame="${inertial_reference_frame}">
-    <origin xyz="0 0 0" rpy="0 0 0" />
-  </xacro:default_chemical_concentration_sensor_macro> -->
-  <!-- <link name="hokuyo_link">
+  <!-- Side scan sonar left -->
+  <xacro:sidescan_sonar namespace="${namespace}" parent_link="${namespace}/base_link" suffix="left">
+    <origin xyz="0.41225 0.1498 -0.04615" rpy="${0.5*pi} ${-5*d2r+pi/3.0} ${0.5*pi}" />
+  </xacro:sidescan_sonar>
+  <!-- Side scan sonar right -->
+  <xacro:sidescan_sonar namespace="${namespace}" parent_link="${namespace}/base_link" suffix="right">
+    <origin xyz="0.41225 -0.1498 -0.04615" rpy="${0.5*pi} ${-5*d2r+pi/3.0} ${-0.5*pi}" />
+  </xacro:sidescan_sonar>
+  <xacro:macro name="forward_multibeam_p900_custom" params="namespace parent_link *origin">
+    <xacro:multibeam_sonar namespace="${namespace}" suffix="" parent_link="${parent_link}" topic="sonar" mass="0.02" update_rate="15" samples="512" fov="1.5708" range_min="1.0" range_max="100.0" range_stddev="0.027" mesh="">
+      <inertia ixx="0.00001" ixy="0.0" ixz="0.0" iyy="0.00001" iyz="0.0" izz="0.00001" />
+      <xacro:insert_block name="origin" />
+      <visual>
+        <geometry>
+          <mesh filename="file://$(find robot-lab)/meshes/p900.dae" scale="1 1 1" />
+        </geometry>
+      </visual>
+    </xacro:multibeam_sonar>
+  </xacro:macro>
+  <xacro:forward_multibeam_p900_custom namespace="${namespace}" parent_link="${namespace}/base_link">
+    <origin xyz="0.45 0.0025 0.19" rpy="0 0 0" />
+  </xacro:forward_multibeam_p900_custom>
+  <link name="${namespace}/depth_sounder">
     <inertial>
       <mass value="0.001" />
@@ -58,5 +40,5 @@
       <origin xyz="0 0 0" rpy="0 0 0" />
       <geometry>
-        <mesh filename="package://robot-lab/meshes/max_sonar_ez4.dae" />
+        <mesh filename="package://robot-lab/meshes/sonar.dae" />
       </geometry>
     </visual>
@@ -64,197 +46,49 @@
       <origin xyz="0 0 0" rpy="0 0 0" />
       <geometry>
-        <box size="0.01 0.01 0.01" />
+        <mesh filename="package://robot-lab/meshes/sonar.dae" />
       </geometry>
     </collision>
-  </link> -->
-  <!-- <link name="side_scan_sonar_right_link">
-    <visual>
-      <origin xyz="0 0 0" rpy="0 0 0" />
-      <geometry>
-        <mesh filename="package://robot-lab/meshes/max_sonar_ez4.dae" />
-      </geometry>
-    </visual>
   </link>
-  <link name="side_scan_sonar_left_link">
-    <visual>
-      <origin xyz="0 0 0" rpy="0 0 0" />
-      <geometry>
-        <mesh filename="package://robot-lab/meshes/max_sonar_ez4.dae" />
-      </geometry>
-    </visual>
-  </link> -->
-  <!-- <link name="camera_link">
-    <collision>
-      <origin xyz="0 0 0" rpy="0 0 0" />
-      <geometry>
-        <mesh filename="package://robot-lab/meshes/flir_a35_housing.stl" />
-      </geometry>
-    </collision>
-    <visual>
-      <origin xyz="0 0 0" rpy="0 0 0" />
-      <geometry>
-        <mesh filename="package://robot-lab/meshes/flir_a35_housing.stl" />
-      </geometry>
-    </visual>
-    <inertial>
-      <mass value="1e-5" />
-      <origin xyz="0 0 0" rpy="0 0 0" />
-      <inertia ixx="1e-6" ixy="0" ixz="0" iyy="1e-6" iyz="0" izz="1e-6" />
-    </inertial>
-  </link> -->
-  <!-- SENSORS -->
-  <!-- <gazebo reference="hokuyo_link">
-    <sensor type="ray" name="head_hokuyo_sensor">
+  <joint name="depth_soundert_joint" type="fixed">
+    <origin xyz="-0.15781 0 0" rpy="0 ${0.5*pi} 0" />
+    <parent link="${namespace}/base_link" />
+    <child link="${namespace}/depth_sounder" />
+  </joint>
+  <gazebo reference="${namespace}/depth_sounder">
+    <sensor type="ray" name="depth_sounder">
       <pose>0 0 0 0 0 0</pose>
+      <update_rate>1</update_rate>
       <visualize>true</visualize>
-      <update_rate>100</update_rate>
       <ray>
         <scan>
           <horizontal>
-            <samples>720</samples>
+            <samples>3</samples>
             <resolution>1</resolution>
-            <min_angle>-2</min_angle>
-            <max_angle>2</max_angle>
+            <min_angle>-0.03</min_angle>
+            <max_angle>0.03</max_angle>
           </horizontal>
+          <vertical>
+            <samples>3</samples>
+            <resolution>1</resolution>
+            <min_angle>-0.03</min_angle>
+            <max_angle>0.03</max_angle>
+          </vertical>
         </scan>
         <range>
-          <min>0.1</min>
-          <max>5.6</max>
+          <min>0.55</min>
+          <max>120</max>
           <resolution>0.01</resolution>
         </range>
-        <noise>
-          <type>gaussian</type>
-          <mean>0.0</mean>
-          <stddev>0.01</stddev>
-        </noise>
       </ray>
-      <plugin name="gazebo_ros_head_hokuyo_controller" filename="libgazebo_ros_laser.so">
-        <topicName>/rrbot/laser/scan</topicName>
-        <frameName>hokuyo_link</frameName>
-      </plugin>
-    </sensor>
-  </gazebo> -->
-  <!-- CAMERA -->
-  <!-- <gazebo reference="camera_link">
-    <sensor type="camera" name="camera1">
-      <update_rate>30.0</update_rate>
-      <camera name="head">
-        <horizontal_fov>1.3962634</horizontal_fov>
-        <image>
-          <width>800</width>
-          <height>800</height>
-          <format>R8G8B8</format>
-        </image>
-        <clip>
-          <near>0.02</near>
-          <far>300</far>
-        </clip>
-        <noise>
-          <type>gaussian</type>
-          <mean>0.0</mean>
-          <stddev>0.007</stddev>
-        </noise>
-      </camera>
-      <plugin name="camera_controller" filename="libgazebo_ros_camera.so">
+      <plugin filename="libgazebo_ros_range.so" name="gazebo_ros_range">
+        <gaussianNoise>0.005</gaussianNoise>
         <alwaysOn>true</alwaysOn>
-        <updateRate>0.0</updateRate>
-        <cameraName>rrbot/camera1</cameraName>
-        <imageTopicName>image_raw</imageTopicName>
-        <cameraInfoTopicName>camera_info</cameraInfoTopicName>
-        <frameName>camera_link</frameName>
-        <hackBaseline>0.07</hackBaseline>
-        <distortionK1>0.0</distortionK1>
-        <distortionK2>0.0</distortionK2>
-        <distortionK3>0.0</distortionK3>
-        <distortionT1>0.0</distortionT1>
-        <distortionT2>0.0</distortionT2>
-      </plugin>
-    </sensor>
-  </gazebo> -->
-  <!-- SIDE SCAN SONAR -->
-  <!-- <gazebo reference="side_scan_sonar_left_link">
-    <sensor type="gpu_ray" name="sonar_left">
-      <pose>0 0 0 0 0 0</pose>
-      <visualize>true</visualize>
-      <update_rate>2</update_rate>
-      <ray>
-        <scan>
-          <horizontal>
-            <samples>60</samples>
-            <resolution>1</resolution>
-            <min_angle>-${0.5*pi/3.0}</min_angle>
-            <max_angle>${0.5*pi/3.0}</max_angle>
-          </horizontal>
-        </scan>
-        <range>
-          <min>1.0</min>
-          <max>200.0</max>
-          <resolution>0.01</resolution>
-        </range>
-        <noise>
-          <type>gaussian</type>
-          <mean>0.0</mean>
-          <stddev>0.027</stddev>
-        </noise>
-      </ray>
-      <plugin name="sonar_left_controller" filename="libgazebo_ros_gpu_laser.so">
-        <topicName>sss_left</topicName>
-        <frameName>side_scan_sonar_left_link</frameName>
+        <updateRate>1</updateRate>
+        <topicName>/depth_sounder_tp</topicName>
+        <frameName>${namespace}/depth_sounder</frameName>
+        <radiation>ultrasound</radiation>
+        <fov>0.06</fov>
       </plugin>
     </sensor>
   </gazebo>
-  <gazebo reference="side_scan_sonar_right_link">
-    <sensor type="gpu_ray" name="sonar_right">
-      <pose>0 0 0 0 0 0</pose>
-      <visualize>true</visualize>
-      <update_rate>2</update_rate>
-      <ray>
-        <scan>
-          <horizontal>
-            <samples>60</samples>
-            <resolution>1</resolution>
-            <min_angle>-${0.5*pi/3.0}</min_angle>
-            <max_angle>${0.5*pi/3.0}</max_angle>
-          </horizontal>
-        </scan>
-        <range>
-          <min>1.0</min>
-          <max>200.0</max>
-          <resolution>0.01</resolution>
-        </range>
-        <noise>
-          <type>gaussian</type>
-          <mean>0.0</mean>
-          <stddev>0.027</stddev>
-        </noise>
-      </ray>
-      <plugin name="sonar_right_controller" filename="libgazebo_ros_gpu_laser.so">
-        <topicName>sss_right</topicName>
-        <frameName>side_scan_sonar_right_link</frameName>
-      </plugin>
-    </sensor>
-  </gazebo> -->
-  <!-- JOINTS -->
-  <!-- <joint name="sonar_joint" type="fixed">
-    <parent link="base_link" />
-    <child link="hokuyo_link" />
-    <origin xyz="0.334 0 0.06" />
-  </joint> -->
-  <!--
-  <joint name="camera_joint" type="fixed">
-    <axis xyz="0 1 0" />
-    <origin xyz="0.25 0 0.12" rpy="0 0 0" />
-    <parent link="base_link" />
-    <child link="camera_link" />
-  </joint> -->
-  <!-- <joint name="sss_right_joint" type="fixed">
-    <origin xyz="-0.0539357 -0.0554493 -0.0530891" rpy="1.570796327 1 -1.570796327" />
-    <parent link="$(arg namespace)/base_link" />
-    <child link="side_scan_sonar_right_link" />
-  </joint>
-  <joint name="sss_left_joint" type="fixed">
-    <origin xyz="-0.0539357 0.0554493 -0.0530891" rpy="1.570796327 1 1.570796327" />
-    <parent link="$(arg namespace)/base_link" />
-    <child link="side_scan_sonar_left_link" />
-  </joint> -->
 </robot>
