Commit message: fix thruster parameters

File: description/urdf/argo_base.xacro (robot description, xacro)
@@ -8,5 +8,4 @@
   <xacro:property name="collision_mesh_file" value="file://$(find robot-lab)/meshes/argo.dae" />
   <xacro:property name="mass" value="28" />
-  <!-- <xacro:property name="mass" value="37.498" /> -->
   <xacro:property name="x_size" value="1.20" />
   <xacro:property name="y_size" value="0.86" />

File: description/urdf/argo_sensors.xacro (robot description, xacro)
@@ -99,5 +99,5 @@
   </xacro:macro>
   <xacro:forward_multibeam_p900_custom namespace="${namespace}" parent_link="${namespace}/base_link">
-    <origin xyz="0.45 0.0025 0.19" rpy="0 0 0" />
+    <origin xyz="0.45 0.0025 0.19" rpy="0 -0.05 0" />
   </xacro:forward_multibeam_p900_custom>
   <link name="${namespace}/depth_sounder">

File: description/urdf/argo_snippets.xacro (robot description, xacro)
@@ -2,5 +2,5 @@
 <robot xmlns:xacro="http://www.ros.org/wiki/xacro">
   <xacro:macro name="thruster_macro" params="namespace thruster_id *origin">
-    <xacro:thruster_module_first_order_basic_fcn_macro namespace="${namespace}" thruster_id="${thruster_id}" mesh_filename="file://$(find robot-lab)/meshes/propeller.dae" dyn_time_constant="0.05" rotor_constant="0.00001">
+    <xacro:thruster_module_first_order_basic_fcn_macro namespace="${namespace}" thruster_id="${thruster_id}" mesh_filename="file://$(find robot-lab)/meshes/propeller.dae" dyn_time_constant="0.05" rotor_constant="0.026546960744430276">
       <xacro:insert_block name="origin" />
     </xacro:thruster_module_first_order_basic_fcn_macro>
