Commit message: fix side scan sonar

File: description/urdf/argo_sensors.xacro (robot description, xacro)
@@ -9,14 +9,84 @@
   <!-- Mount a Pose 3D sensor. -->
   <xacro:default_pose_3d_macro namespace="${namespace}" parent_link="${namespace}/base_link" inertial_reference_frame="${inertial_reference_frame}" />
+  <xacro:macro name="argo_multibeam_sonar" params="namespace suffix parent_link topic mass update_rate
+  samples fov range_min range_max range_stddev mesh
+  *inertia *origin *visual">
+    <!-- Sensor link -->
+    <link name="${namespace}/sonar${suffix}_link">
+      <inertial>
+        <xacro:insert_block name="inertia" />
+        <mass value="${mass}" />
+        <origin xyz="0 0 0" rpy="0 0 0" />
+      </inertial>
+      <xacro:insert_block name="visual" />
+      <xacro:no_collision />
+    </link>
+    <joint name="${namespace}_sonar${suffix}_joint" type="revolute">
+      <xacro:insert_block name="origin" />
+      <parent link="${parent_link}" />
+      <child link="${namespace}/sonar${suffix}_link" />
+      <limit upper="0" lower="0" effort="0" velocity="0" />
+      <axis xyz="1 0 0" />
+    </joint>
+    <gazebo reference="${namespace}/sonar${suffix}_link">
+      <sensor type="gpu_ray" name="sonar${suffix}">
+        <pose>0 0 0 0 0 0</pose>
+        <visualize>true</visualize>
+        <update_rate>${update_rate}</update_rate>
+        <ray>
+          <scan>
+            <horizontal>
+              <samples>${samples}</samples>
+              <resolution>1</resolution>
+              <min_angle>-${0.5*fov}</min_angle>
+              <max_angle>${0.5*fov}</max_angle>
+            </horizontal>
+          </scan>
+          <range>
+            <min>${range_min}</min>
+            <max>${range_max}</max>
+            <resolution>0.01</resolution>
+          </range>
+          <noise>
+            <type>gaussian</type>
+            <mean>0.0</mean>
+            <stddev>${range_stddev}</stddev>
+          </noise>
+        </ray>
+        <plugin name="sonar${suffix}_controller" filename="libgazebo_ros_gpu_laser.so">
+          <topicName>${topic}</topicName>
+          <frameName>sonar${suffix}_link</frameName>
+        </plugin>
+        <!-- TODO: Separate switchable sonar version in another macro -->
+        <!-- <plugin name="switchable_sonar{suffix}_ros_interface" filename="libuuv_gazebo_ros_switchable_gpu_ray_sensor.so">
+      <namespace>${namespace}</namespace>
+      <input_topic>${topic}</input_topic>
+  </plugin> -->
+      </sensor>
+    </gazebo>
+  </xacro:macro>
+  <!-- Side scan sonar -->
+  <xacro:macro name="argo_sidescan_sonar" params="namespace parent_link suffix *origin">
+    <xacro:argo_multibeam_sonar namespace="${namespace}" suffix="${suffix}" parent_link="${parent_link}" topic="sss_${suffix}" mass="0.015" update_rate="2" samples="60" fov="${pi/3.0}" range_min="1.0" range_max="200.0" range_stddev="0.027" mesh="">
+      <inertia ixx="0.00001" ixy="0.0" ixz="0.0" iyy="0.00001" iyz="0.0" izz="0.00001" />
+      <xacro:insert_block name="origin" />
+      <visual>
+        <origin xyz="0 0 0" rpy="0 0 0" />
+        <geometry>
+          <box size="0.001 0.001 0.001" />
+        </geometry>
+      </visual>
+    </xacro:argo_multibeam_sonar>
+  </xacro:macro>
   <!-- Side scan sonar left -->
-  <xacro:sidescan_sonar namespace="${namespace}" parent_link="${namespace}/base_link" suffix="left">
+  <xacro:argo_sidescan_sonar namespace="${namespace}" parent_link="${namespace}/base_link" suffix="left">
     <origin xyz="0.41225 0.1498 -0.04615" rpy="${0.5*pi} ${-5*d2r+pi/3.0} ${0.5*pi}" />
-  </xacro:sidescan_sonar>
+  </xacro:argo_sidescan_sonar>
   <!-- Side scan sonar right -->
-  <xacro:sidescan_sonar namespace="${namespace}" parent_link="${namespace}/base_link" suffix="right">
+  <xacro:argo_sidescan_sonar namespace="${namespace}" parent_link="${namespace}/base_link" suffix="right">
     <origin xyz="0.41225 -0.1498 -0.04615" rpy="${0.5*pi} ${-5*d2r+pi/3.0} ${-0.5*pi}" />
-  </xacro:sidescan_sonar>
+  </xacro:argo_sidescan_sonar>
   <xacro:macro name="forward_multibeam_p900_custom" params="namespace parent_link *origin">
-    <xacro:multibeam_sonar namespace="${namespace}" suffix="" parent_link="${parent_link}" topic="sonar" mass="0.02" update_rate="15" samples="512" fov="1.5708" range_min="1.0" range_max="100.0" range_stddev="0.027" mesh="">
+    <xacro:argo_multibeam_sonar namespace="${namespace}" suffix="" parent_link="${parent_link}" topic="sonar" mass="0.02" update_rate="15" samples="512" fov="1.5708" range_min="1.0" range_max="100.0" range_stddev="0.027" mesh="">
       <inertia ixx="0.00001" ixy="0.0" ixz="0.0" iyy="0.00001" iyz="0.0" izz="0.00001" />
       <xacro:insert_block name="origin" />
@@ -26,5 +96,5 @@
         </geometry>
       </visual>
-    </xacro:multibeam_sonar>
+    </xacro:argo_multibeam_sonar>
   </xacro:macro>
   <xacro:forward_multibeam_p900_custom namespace="${namespace}" parent_link="${namespace}/base_link">

Commit message: fix

File: description/urdf/argo_sensors.xacro (robot description, xacro)
@@ -30,5 +30,5 @@
     </joint>
     <gazebo reference="${namespace}/sonar${suffix}_link">
-      <sensor type="gpu_ray" name="sonar${suffix}">
+      <sensor type="ray" name="sonar${suffix}">
         <pose>0 0 0 0 0 0</pose>
         <visualize>true</visualize>
@@ -54,5 +54,5 @@
           </noise>
         </ray>
-        <plugin name="sonar${suffix}_controller" filename="libgazebo_ros_gpu_laser.so">
+        <plugin name="sonar${suffix}_controller" filename="libgazebo_ros_laser.so">
           <topicName>${topic}</topicName>
           <frameName>sonar${suffix}_link</frameName>
@@ -88,5 +88,5 @@
   </xacro:argo_sidescan_sonar>
   <xacro:macro name="forward_multibeam_p900_custom" params="namespace parent_link *origin">
-    <xacro:argo_multibeam_sonar namespace="${namespace}" suffix="" parent_link="${parent_link}" topic="sonar" mass="0.02" update_rate="15" samples="512" fov="1.5708" range_min="1.0" range_max="30.0" range_stddev="0.027" mesh="">
+    <xacro:argo_multibeam_sonar namespace="${namespace}" suffix="" parent_link="${parent_link}" topic="sonar" mass="0.02" update_rate="100" samples="720" fov="4" range_min="0.5" range_max="5.6" range_stddev="0.01" mesh="">
       <inertia ixx="0.00001" ixy="0.0" ixz="0.0" iyy="0.00001" iyz="0.0" izz="0.00001" />
       <xacro:insert_block name="origin" />
@@ -99,5 +99,5 @@
   </xacro:macro>
   <xacro:forward_multibeam_p900_custom namespace="${namespace}" parent_link="${namespace}/base_link">
-    <origin xyz="0.45 0.0025 0.19" rpy="0 -0.05 0" />
+    <origin xyz="0.45 0.0025 0.19" rpy="0 0 0" />
   </xacro:forward_multibeam_p900_custom>
   <link name="${namespace}/depth_sounder">
