Commit message: thrusters mounting

File: description/robots/argo_default.xacro (robot description, xacro)
@@ -16,9 +16,4 @@
     </gazebo>
   </xacro:argo_base>
-  <!-- <gazebo>
-    <plugin name="BuoyancyPlugin" filename="libBuoyancyPlugin.so">
-      <fluid_density>1000</fluid_density>
-    </plugin>
-  </gazebo> -->
   <xacro:default_joint_state_publisher namespace="$(arg namespace)" update_rate="50" />
 </robot>

File: description/urdf/argo.gazebo.xacro (robot description, xacro)
@@ -1,34 +1,37 @@
 <?xml version="1.0"?>
 <robot xmlns:xacro="http://www.ros.org/wiki/xacro">
-    <xacro:property name="cob" value="0.0 0.0 0.3" />
-    <xacro:property name="volume" value="1.83826" />
-    <xacro:macro name="argo_hydro_model" params="namespace">
-        <link name="${namespace}/base_link">
-            <neutrally_buoyant>0</neutrally_buoyant>
-            <volume>${volume}</volume>
-            <box>
-                <width>1.5</width>
-                <length>2.6</length>
-                <height>1.6</height>
-            </box>
-            <center_of_buoyancy>${cob}</center_of_buoyancy>
-            <hydrodynamic_model>
-                <type>fossen</type>
-                <added_mass>
-                     779.79 -6.8773 -103.32  8.5426 -165.54 -7.8033
-                    -6.8773    1222   51.29  409.44 -5.8488  62.726
-                    -103.32   51.29  3659.9  6.1112 -386.42  10.774
-                     8.5426  409.44  6.1112   534.9 -10.027  21.019
-                    -165.54 -5.8488 -386.42 -10.027  842.69 -1.1162
-                    -7.8033  62.726  10.775  21.019 -1.1162  224.32
-                </added_mass>
-                <linear_damping>
-                    -74.82 -69.48 -728.4 -268.8 -309.77 -105
-                </linear_damping>
-                <quadratic_damping>
-                    -748.22 -992.53 -1821.01 -672 -774.44 -523.27
-                </quadratic_damping>
-            </hydrodynamic_model>
-        </link>
-    </xacro:macro>
+  <xacro:property name="cob" value="0 0 0.155" />
+  <xacro:property name="volume" value="0.2668" />
+  <xacro:property name="x_size" value="1.2" />
+  <xacro:property name="y_size" value="0.86" />
+  <xacro:property name="z_size" value="0.6" />
+  <xacro:macro name="argo_hydro_model" params="namespace">
+    <link name="${namespace}/base_link">
+      <neutrally_buoyant>1</neutrally_buoyant>
+      <volume>${volume}</volume>
+      <box>
+        <width>${y_size}</width>
+        <length>${x_size}</length>
+        <height>${z_size}</height>
+      </box>
+      <center_of_buoyancy>${cob}</center_of_buoyancy>
+      <hydrodynamic_model>
+        <type>fossen</type>
+        <added_mass>
+          1.7182 0 0 0 0 0
+          0 0 0 0 0 0
+          0 0 5.468 0 0 0
+          0 0 0 0 0 0
+          0 0 0 0 1.2481 0
+          0 0 0 0 0 0.4006
+        </added_mass>
+        <linear_damping>
+          -11.7391 -20 -31.8678 -25 -44.9085 -5
+        </linear_damping>
+        <quadratic_damping>
+          0 0 0 0 0 0
+        </quadratic_damping>
+      </hydrodynamic_model>
+    </link>
+  </xacro:macro>
 </robot>

File: description/urdf/argo_actuators.xacro (robot description, xacro)
@@ -1,9 +1,12 @@
 <?xml version="1.0"?>
-<robot xmlns:xacro="http://www.ros.org/wiki/xacro" >
+<robot xmlns:xacro="http://www.ros.org/wiki/xacro">
+  <xacro:thruster_macro namespace="${namespace}" thruster_id="0">
+    <origin xyz="-0.088 -0.1192 -0.0061828" rpy="0 0 ${pi}" />
+  </xacro:thruster_macro>
   <xacro:thruster_macro namespace="${namespace}" thruster_id="1">
-    <origin xyz="-0.068067 0.0585 -0.076978" rpy="0 0 ${pi}"/>
+    <origin xyz="-0.088 0.1192 -0.0061828" rpy="0 0 ${pi}" />
   </xacro:thruster_macro>
   <xacro:thruster_macro namespace="${namespace}" thruster_id="2">
-    <origin xyz="-0.068067 -0.0585 -0.076978" rpy="0 0 ${pi}"/>
+    <origin xyz="0.067 0 0.1258172" rpy="0 -${0.5*pi} 0" />
   </xacro:thruster_macro>
 </robot>

File: description/urdf/argo_base.xacro (robot description, xacro)
@@ -5,13 +5,20 @@
   <xacro:include filename="$(find robot-lab)/description/urdf/argo_snippets.xacro" />
   <xacro:include filename="$(find uuv_gazebo_ros_plugins)/urdf/snippets.xacro" />
-  <xacro:property name="visual_mesh_file" value="file://$(find robot-lab)/meshes/robot.dae" />
-  <xacro:property name="mass" value="1862.87" />
+  <xacro:property name="visual_mesh_file" value="file://$(find robot-lab)/meshes/argo.dae" />
+  <xacro:property name="collision_mesh_file" value="file://$(find robot-lab)/meshes/argo.dae" />
+  <xacro:property name="mass" value="28" />
   <!-- <xacro:property name="mass" value="37.498" /> -->
+  <xacro:property name="x_size" value="1.20" />
+  <xacro:property name="y_size" value="0.86" />
+  <xacro:property name="z_size" value="0.6" />
   <xacro:macro name="argo_base" params="namespace *gazebo inertial_reference_frame">
+    <gazebo reference="${namespace}/base_link">
+      <selfCollide>false</selfCollide>
+    </gazebo>
     <link name="${namespace}/base_link">
       <inertial>
         <mass value="${mass}" />
         <origin xyz="0 0 0" rpy="0 0 0" />
-        <inertia ixx="525.39" ixy="1.44" ixz="33.41" iyy="794.20" iyz="2.6" izz="691.23" />
+        <inertia ixx="${0.2*mass*y_size*y_size + 0.2*mass*z_size*z_size}" ixy="0.0" ixz="0.0" iyy="${0.2*mass*x_size*x_size + 0.2*mass*z_size*z_size}" iyz="0.0" izz="${0.2*mass*x_size*x_size + 0.2*mass*y_size*y_size}" />
       </inertial>
       <visual>
@@ -24,5 +31,5 @@
         <origin rpy="0 0 0" xyz="0 0 0" />
         <geometry>
-          <mesh filename="${visual_mesh_file}" scale="1 1 1" />
+          <mesh filename="${collision_mesh_file}" scale="1 1 1" />
         </geometry>
       </collision>

File: description/urdf/argo_sensors.xacro (robot description, xacro)
@@ -1,4 +1,16 @@
 <?xml version="1.0"?>
 <robot xmlns:xacro="http://www.ros.org/wiki/xacro">
+  <!-- Mount a GPS. -->
+  <xacro:default_gps namespace="${namespace}" parent_link="${namespace}/base_link" />
+  <!-- Mount a Pose 3D sensor. -->
+  <xacro:default_pose_3d_macro namespace="${namespace}" parent_link="${namespace}/base_link" inertial_reference_frame="${inertial_reference_frame}" />
+  <!-- IMU  -->
+  <xacro:default_imu_macro namespace="${namespace}" parent_link="${namespace}/base_link" inertial_reference_frame="${inertial_reference_frame}">
+    <origin xyz="0 0 0" rpy="0 0 0" />
+  </xacro:default_imu_macro>
+  <!-- Add a chemical particle concentration sensor -->
+  <xacro:default_chemical_concentration_sensor namespace="${namespace}" parent_link="${namespace}/base_link">
+    <origin xyz="0 0 0" rpy="0 0 0" />
+  </xacro:default_chemical_concentration_sensor>
   <!-- DVL  -->
   <!-- <xacro:default_dvl_macro namespace="${namespace}" parent_link="${namespace}/base_link" inertial_reference_frame="${inertial_reference_frame}">
@@ -32,5 +44,5 @@
   <!-- <xacro:default_gps namespace="${namespace}" parent_link="${namespace}/base_link" /> -->
   <!-- Mount a Pose 3D sensor. -->
-  <xacro:default_pose_3d_macro namespace="${namespace}" parent_link="${namespace}/base_link" inertial_reference_frame="${inertial_reference_frame}" />
+  <!-- <xacro:default_pose_3d_macro namespace="${namespace}" parent_link="${namespace}/base_link" inertial_reference_frame="${inertial_reference_frame}" /> -->
   <!-- Mount chemical particle concentration sensor -->
   <!-- <xacro:default_chemical_concentration_sensor_macro namespace="${namespace}" parent_link="${namespace}/base_link" inertial_reference_frame="${inertial_reference_frame}">

File: description/urdf/argo_snippets.xacro (robot description, xacro)
@@ -2,5 +2,5 @@
 <robot xmlns:xacro="http://www.ros.org/wiki/xacro">
   <xacro:macro name="thruster_macro" params="namespace thruster_id *origin">
-    <xacro:thruster_module_first_order_basic_fcn_macro namespace="${namespace}" thruster_id="${thruster_id}" mesh_filename="file://$(find robot-lab)/meshes/propeller.dae" dyn_time_constant="0.05" rotor_constant="0.026546960744430276">
+    <xacro:thruster_module_first_order_basic_fcn_macro namespace="${namespace}" thruster_id="${thruster_id}" mesh_filename="file://$(find robot-lab)/meshes/propeller.dae" dyn_time_constant="0.05" rotor_constant="0.00001">
       <xacro:insert_block name="origin" />
     </xacro:thruster_module_first_order_basic_fcn_macro>

Commit message: add README

File: description/robots/argo_default.xacro (robot description, xacro)
@@ -4,6 +4,6 @@
   <xacro:arg name="namespace" default="argo" />
   <xacro:arg name="inertial_reference_frame" default="world" />
-  <xacro:include filename="$(find robot-lab)/description/urdf/argo_base.xacro" />
-  <xacro:include filename="$(find robot-lab)/description/urdf/argo.gazebo.xacro" />
+  <xacro:include filename="$(find digital-twin)/description/urdf/argo_base.xacro" />
+  <xacro:include filename="$(find digital-twin)/description/urdf/argo.gazebo.xacro" />
   <xacro:argo_base namespace="$(arg namespace)" inertial_reference_frame="$(arg inertial_reference_frame)">
     <gazebo>

File: description/urdf/argo_base.xacro (robot description, xacro)
@@ -3,8 +3,8 @@
   <xacro:include filename="$(find uuv_descriptions)/urdf/common.urdf.xacro" />
   <xacro:include filename="$(find uuv_sensor_ros_plugins)/urdf/sensor_snippets.xacro" />
-  <xacro:include filename="$(find robot-lab)/description/urdf/argo_snippets.xacro" />
+  <xacro:include filename="$(find digital-twin)/description/urdf/argo_snippets.xacro" />
   <xacro:include filename="$(find uuv_gazebo_ros_plugins)/urdf/snippets.xacro" />
-  <xacro:property name="visual_mesh_file" value="file://$(find robot-lab)/meshes/argo.dae" />
-  <xacro:property name="collision_mesh_file" value="file://$(find robot-lab)/meshes/argo.dae" />
+  <xacro:property name="visual_mesh_file" value="file://$(find digital-twin)/meshes/argo.dae" />
+  <xacro:property name="collision_mesh_file" value="file://$(find digital-twin)/meshes/argo.dae" />
   <xacro:property name="mass" value="28" />
   <xacro:property name="x_size" value="1.20" />
@@ -35,6 +35,6 @@
     </link>
     <xacro:insert_block name="gazebo" />
-    <xacro:include filename="$(find robot-lab)/description/urdf/argo_sensors.xacro" />
-    <xacro:include filename="$(find robot-lab)/description/urdf/argo_actuators.xacro" />
+    <xacro:include filename="$(find digital-twin)/description/urdf/argo_sensors.xacro" />
+    <xacro:include filename="$(find digital-twin)/description/urdf/argo_actuators.xacro" />
   </xacro:macro>
 </robot>

File: description/urdf/argo_sensors.xacro (robot description, xacro)
@@ -93,5 +93,5 @@
       <visual>
         <geometry>
-          <mesh filename="file://$(find robot-lab)/meshes/p900.dae" scale="1 1 1" />
+          <mesh filename="file://$(find digital-twin)/meshes/p900.dae" scale="1 1 1" />
         </geometry>
       </visual>
@@ -110,5 +110,5 @@
       <origin xyz="0 0 0" rpy="0 0 0" />
       <geometry>
-        <mesh filename="package://robot-lab/meshes/sonar.dae" />
+        <mesh filename="package://digital-twin/meshes/sonar.dae" />
       </geometry>
     </visual>
@@ -116,5 +116,5 @@
       <origin xyz="0 0 0" rpy="0 0 0" />
       <geometry>
-        <mesh filename="package://robot-lab/meshes/sonar.dae" />
+        <mesh filename="package://digital-twin/meshes/sonar.dae" />
       </geometry>
     </collision>

File: description/urdf/argo_snippets.xacro (robot description, xacro)
@@ -2,5 +2,5 @@
 <robot xmlns:xacro="http://www.ros.org/wiki/xacro">
   <xacro:macro name="thruster_macro" params="namespace thruster_id *origin">
-    <xacro:thruster_module_first_order_basic_fcn_macro namespace="${namespace}" thruster_id="${thruster_id}" mesh_filename="file://$(find robot-lab)/meshes/propeller.dae" dyn_time_constant="0.05" rotor_constant="0.026546960744430276">
+    <xacro:thruster_module_first_order_basic_fcn_macro namespace="${namespace}" thruster_id="${thruster_id}" mesh_filename="file://$(find digital-twin)/meshes/propeller.dae" dyn_time_constant="0.05" rotor_constant="0.026546960744430276">
       <xacro:insert_block name="origin" />
     </xacro:thruster_module_first_order_basic_fcn_macro>
